Commit message: feat[urdf]: created urdf and launched

File: install/scout_description/share/scout_description/urdf/scout_v2.xacro (robot description, xacro)
@@ -1 +1 @@
-/mnt/toshiba_hdd/code/robot-learning/dlrl/biolab-isaacsim_ws/src/scout_ros/scout_description/urdf/scout_v2.xacro
+/mnt/toshiba_hdd/code/robot-learning/dlrl/biolab-isaacsim_ws/src/scout/scout_description/urdf/scout_v2.xacro

File: install/scout_description/share/scout_description/urdf/scout_wheel_type1.xacro (robot description, xacro)
@@ -1 +1 @@
-/mnt/toshiba_hdd/code/robot-learning/dlrl/biolab-isaacsim_ws/src/scout_ros/scout_description/urdf/scout_wheel_type1.xacro
+/mnt/toshiba_hdd/code/robot-learning/dlrl/biolab-isaacsim_ws/src/scout/scout_description/urdf/scout_wheel_type1.xacro

File: install/scout_description/share/scout_description/urdf/scout_wheel_type2.xacro (robot description, xacro)
@@ -1 +1 @@
-/mnt/toshiba_hdd/code/robot-learning/dlrl/biolab-isaacsim_ws/src/scout_ros/scout_description/urdf/scout_wheel_type2.xacro
+/mnt/toshiba_hdd/code/robot-learning/dlrl/biolab-isaacsim_ws/src/scout/scout_description/urdf/scout_wheel_type2.xacro

File: src/scout_with_piper_description/urdf/piper_description.xacro (robot description, xacro)
@@ -1,4 +1,6 @@
 <?xml version="1.0" encoding="utf-8"?>
 <robot name="piper" xmlns:xacro="http://ros.org/wiki/xacro">
+<xacro:arg name="left_camera_xyz" default="0 0 0" />
+<xacro:arg name="left_camera_rpy" default="0 0 0" />
 <!-- arm: agx_arm_urdf/piper (official DAE visuals, link names prefixed) -->
 <link name="piper_base_link">>
@@ -283,4 +285,32 @@
     <axis xyz="0 1 0" />
     <limit lower="0" upper="0.05" effort="100" velocity="5" />
+  </joint>
+  <!-- Left camera mounted on the gripper base -->
+  <link name="left_camera_link">
+    <inertial>
+      <origin xyz="0 0 0" rpy="0 0 0" />
+      <mass value="0.05" />
+      <inertia ixx="0.00001" ixy="0" ixz="0" iyy="0.00001" iyz="0" izz="0.00001" />
+    </inertial>
+    <visual>
+      <origin xyz="0 0 0" rpy="0 0 0" />
+      <geometry>
+        <box size="0.02 0.02 0.02" />
+      </geometry>
+      <material name="camera_grey">
+        <color rgba="0.2 0.2 0.2 1" />
+      </material>
+    </visual>
+    <collision>
+      <origin xyz="0 0 0" rpy="0 0 0" />
+      <geometry>
+        <box size="0.02 0.02 0.02" />
+      </geometry>
+    </collision>
+  </link>
+  <joint name="left_camera_joint" type="fixed">
+    <origin xyz="$(arg left_camera_xyz)" rpy="$(arg left_camera_rpy)" />
+    <parent link="gripper_base_link" />
+    <child link="left_camera_link" />
   </joint>
 <!-- controller -->
