Commit message: chores[git]: cleanup and update gitignore

File: src/scout_with_piper_description/urdf/lift_actuator.xacro (robot description, xacro)
@@ -146,5 +146,4 @@
       <axis xyz="0 0 1" />
       <limit lower="0" upper="${lift_travel}" effort="500" velocity="0.05" />
-      <dynamics damping="1000" friction="10" />
     </joint>
   </xacro:macro>

File: src/scout_with_piper_description/urdf/lift_actuator_small.xacro (robot description, xacro)
@@ -146,5 +146,4 @@
       <axis xyz="0 0 1" />
       <limit lower="0" upper="${lift_travel}" effort="500" velocity="0.05" />
-      <dynamics damping="1000" friction="10" />
     </joint>
   </xacro:macro>

File: src/scout_with_piper_description/urdf/piper_description.xacro (robot description, xacro)
@@ -287,5 +287,5 @@
   </joint>
   <!-- Left camera mounted on the gripper base -->
-  <link name="left_camera_link">
+  <link name="gripper_left_camera_link">
     <inertial>
       <origin xyz="0 0 0" rpy="0 0 0" />
@@ -309,8 +309,8 @@
     </collision>
   </link>
-  <joint name="left_camera_joint" type="fixed">
+  <joint name="gripper_left_camera_joint" type="fixed">
     <origin xyz="$(arg left_camera_xyz)" rpy="$(arg left_camera_rpy)" />
     <parent link="gripper_base_link" />
-    <child link="left_camera_link" />
+    <child link="gripper_left_camera_link" />
   </joint>
 <!-- controller -->

File: src/scout_with_piper_description/urdf/scout_mini_piper.urdf (robot description, URDF)
Before this commit: robot scout_mini_piper, 19 links, 18 joints
Links:
- removed link left_camera_link
- added link gripper_left_camera_link, mass 0.05; collision box size=0.02 0.02 0.02; visual box size=0.02 0.02 0.02
Joints:
- removed joint left_camera_joint
- added joint gripper_left_camera_joint: type fixed, parent gripper_base_link, child gripper_left_camera_link, origin xyz=0 0 0 rpy=0 0 0
