Commit message: fix[urdf]: remove root inertia so robot_state_publisher publishes TF

File: src/scout_with_piper_description/urdf/piper_description.xacro (robot description, xacro)
@@ -313,4 +313,17 @@
     <parent link="gripper_base_link" />
     <child link="gripper_left_camera_link" />
+  </joint>
+  <!-- Optical frame (REP-103): x right, y down, z forward -->
+  <link name="gripper_left_camera_optical_link">
+    <inertial>
+      <origin xyz="0 0 0" rpy="0 0 0" />
+      <mass value="0.001" />
+      <inertia ixx="1e-06" ixy="0" ixz="0" iyy="1e-06" iyz="0" izz="1e-06" />
+    </inertial>
+  </link>
+  <joint name="gripper_left_camera_optical_joint" type="fixed">
+    <origin xyz="0 0 0" rpy="-1.5708 0 -1.5708" />
+    <parent link="gripper_left_camera_link" />
+    <child link="gripper_left_camera_optical_link" />
   </joint>
 <!-- controller -->

File: src/scout_with_piper_description/urdf/scout_mini.xacro (robot description, xacro)
@@ -15,9 +15,4 @@
       </geometry>
     </collision>
-    <inertial>
-      <mass value="60"/>
-      <origin xyz="0.0 0.0 0.0"/>
-      <inertia ixx="2.288641" ixy="0" ixz="0" iyy="5.103976" iyz="0" izz="3.431465"/>
-    </inertial>
   </link>
   <link name="inertial_link">

File: src/scout_with_piper_description/urdf/scout_mini_piper.urdf (robot description, URDF)
Before this commit: robot scout_mini_piper, 19 links, 18 joints
Links:
- added link gripper_left_camera_optical_link, mass 0.001
- link base_link: mass 60 -> None
Joints:
- added joint gripper_left_camera_optical_joint: type fixed, parent gripper_left_camera_link, child gripper_left_camera_optical_link, origin xyz=0 0 0 rpy=-1.5708 0 -1.5708
