Commit message: fix[urdf]: restore base inertia via base_footprint root link

File: src/scout_with_piper_description/urdf/scout_mini.xacro (robot description, xacro)
@@ -2,4 +2,10 @@
 <robot name="scout_mini" xmlns:xacro="http://ros.org/wiki/xacro">
   <!-- Scout Mini base with indoor wheels (wheel.dae), not the rugged type1/type2 wheels. -->
+  <link name="base_footprint"/>
+  <joint name="base_footprint_joint" type="fixed">
+    <parent link="base_footprint"/>
+    <child link="base_link"/>
+    <origin xyz="0 0 0" rpy="0 0 0"/>
+  </joint>
   <link name="base_link">
     <visual>
@@ -15,4 +21,9 @@
       </geometry>
     </collision>
+    <inertial>
+      <mass value="60"/>
+      <origin xyz="0.0 0.0 0.0"/>
+      <inertia ixx="2.288641" ixy="0" ixz="0" iyy="5.103976" iyz="0" izz="3.431465"/>
+    </inertial>
   </link>
   <link name="inertial_link">

File: src/scout_with_piper_description/urdf/scout_mini_piper.urdf (robot description, URDF)
Before this commit: robot scout_mini_piper, 20 links, 19 joints
Links:
- added link base_footprint
- link base_link: mass None -> 60
Joints:
- added joint base_footprint_joint: type fixed, parent base_footprint, child base_link, origin xyz=0 0 0 rpy=0 0 0

Commit message: fix[urdf]: remove base_footprint root link for Isaac Sim

File: src/scout_with_piper_description/urdf/scout_mini.xacro (robot description, xacro)
@@ -2,10 +2,4 @@
 <robot name="scout_mini" xmlns:xacro="http://ros.org/wiki/xacro">
   <!-- Scout Mini base with indoor wheels (wheel.dae), not the rugged type1/type2 wheels. -->
-  <link name="base_footprint"/>
-  <joint name="base_footprint_joint" type="fixed">
-    <parent link="base_footprint"/>
-    <child link="base_link"/>
-    <origin xyz="0 0 0" rpy="0 0 0"/>
-  </joint>
   <link name="base_link">
     <visual>

File: src/scout_with_piper_description/urdf/scout_mini_piper.urdf (robot description, URDF)
Before this commit: robot scout_mini_piper, 21 links, 20 joints
Links:
- removed link base_footprint
Joints:
- removed joint base_footprint_joint

File: src/scout_with_piper_description/urdf/scout_piper.urdf (robot description, URDF)
Before this commit: robot scout_piper, 20 links, 19 joints
Joints:
- joint base_footprint_joint: child base_footprint -> base_link; origin xyz=0 0 -0.23479 rpy=0 0 0 -> xyz=0 0 0.23479 rpy=0 0 0; parent base_link -> base_footprint

File: src/scout_with_piper_description/urdf/scout_v2.xacro (robot description, xacro)
@@ -39,7 +39,7 @@
     <link name="base_footprint"/>
     <joint name="base_footprint_joint" type="fixed">
-        <origin xyz="0 0 ${wheel_vertical_offset - wheel_radius}" rpy="0 0 0" />
-        <parent link="base_link" />
-        <child link="base_footprint" />
+        <origin xyz="0 0 ${wheel_radius - wheel_vertical_offset}" rpy="0 0 0" />
+        <parent link="base_footprint" />
+        <child link="base_link" />
     </joint>
     <link name="inertial_link">

Commit message: fix[nav]: integrate collision_monitor config

File: src/scout_with_piper_description/urdf/scout_mini.xacro (robot description, xacro)
@@ -15,9 +15,9 @@
       </geometry>
     </collision>
-    <inertial>
-      <mass value="60"/>
-      <origin xyz="0.0 0.0 0.0"/>
-      <inertia ixx="2.288641" ixy="0" ixz="0" iyy="5.103976" iyz="0" izz="3.431465"/>
-    </inertial>
+    <!-- <inertial> -->
+    <!--   <mass value="60"/> -->
+    <!--   <origin xyz="0.0 0.0 0.0"/> -->
+    <!--   <inertia ixx="2.288641" ixy="0" ixz="0" iyy="5.103976" iyz="0" izz="3.431465"/> -->
+    <!-- </inertial> -->
   </link>
   <link name="inertial_link">
